File: KBD8X-MK2.sch (KiCad schematic (older format))
At the start: 22 parts, among them J1 AVR-ISP-6, Q1 DSS60601MZ4-13, SW1 SW_Push, U1 ATmega32U4-MU, U2 PRTR5V0U2X, Y1 16MHz

Commit message: Add top reset switch & more warning text
Parts:
- added SW4: SW_Push, random-keyboard-parts:SKQG-1155865, symbol Switch:SW_Push
- J1: symbol Connector:AVR-ISP-6 -> KBD8X-MK2-rescue:AVR-ISP-6-Connector
- U1: symbol MCU_Microchip_ATmega:ATmega32U4-MU -> KBD8X-MK2-rescue:ATmega32U4-MU-MCU_Microchip_ATmega
Connections:
- wire segments 81 -> 83
Changed lines of the file:
@@
 EESchema Schematic File Version 4
-LIBS:Voyager87-cache
-EELAYER 26 0
+EELAYER 30 0
 EELAYER END
 $Descr A4 11693 8268
@@
 	1650 5375 1650 5425
 $Comp
-L Connector:AVR-ISP-6 J1
+L KBD8X-MK2-rescue:AVR-ISP-6-Connector J1
 U 1 1 5B68D1BE
 P 4475 1725
@@
 Wire Wire Line
 	1550 2475 1700 2475
-$Comp
-L Switch:SW_Push SW1
-U 1 1 5C4DB62B
-P 3450 3550
-F 0 "SW1" H 3450 3835 50  0000 C CNN
-F 1 "SW_Push" H 3450 3744 50  0000 C CNN
-F 2 "random-keyboard-parts:SKQG-1155865" H 3450 3750 50  0001 C CNN
-F 3 "" H 3450 3750 50  0001 C CNN
-	1    3450 3550
-	1    0    0    -1
-$EndComp
 Wire Wire Line
 	3650 3550 3775 3550
@@
 RGBLED
 $Comp
-L MCU_Microchip_ATmega:ATmega32U4-MU U1
+L KBD8X-MK2-rescue:ATmega32U4-MU-MCU_Microchip_ATmega U1
 U 1 1 618B6D6D
 P 4800 5050
@@
 Text GLabel 4875 1525 2    50   Input ~ 0
 RGBLED
+$Comp
+L Switch:SW_Push SW1
+U 1 1 5C4DB62B
+P 3450 3550
+F 0 "SW1" H 3450 3835 50  0000 C CNN
+F 1 "SW_Push" H 3450 3744 50  0000 C CNN
+F 2 "random-keyboard-parts:SKQG-1155865" H 3450 3750 50  0001 C CNN
+F 3 "" H 3450 3750 50  0001 C CNN
+	1    3450 3550
+	1    0    0    -1
+$EndComp
+$Comp
+L Switch:SW_Push SW4
+U 1 1 5E8C2545
+P 3450 3650
+F 0 "SW4" H 3450 3935 50  0000 C CNN
+F 1 "SW_Push" H 3450 3844 50  0000 C CNN
+F 2 "random-keyboard-parts:SKQG-1155865" H 3450 3850 50  0001 C CNN
+F 3 "" H 3450 3850 50  0001 C CNN
+	1    3450 3650
+	-1   0    0    1
+$EndComp
+Wire Wire Line
+	3650 3550 3650 3650
+Connection ~ 3650 3550
+Wire Wire Line
+	3250 3550 3250 3650
+Connection ~ 3250 3550
 $EndSCHEMATC
